File: Placa/_autosave-prueba1.kicad_pcb (KiCad board)
At the start: 2 copper layers, 74.9 x 63.5 mm, 29 parts

Commit message: Commit Prueba Archivos Placa
Parts:
- removed +3: C8051F352, TQFP32
- removed 0,1micF1: C8, SM1206
- removed 0,1micF2: C9, SM1206
- removed 0,1micF3: C12, SM1206
- removed 0,1micF4: C10, SM1206
- removed 0,1micF5: C11, SM1206
- removed ??1: MAX232_TID, DIP-16__300
- removed C1, C2, C3, C4, C5, C6, C7, C8: 0,1micF, SM1206
- removed JP1, JP2, JP3, JP4, JP5, JP6: JUMPER, PINHEAD1-2
- removed R1, R2, R3, R4, R5, R6, R7, R8: 100ohm, SM1206
Other:
- board outline removed
