File: Placa/PPS1.kicad_pcb.kicad_pcb (KiCad board)
At the start: 2 copper layers, 106.2 x 66.5 mm, 54 parts, among them J1 JACK_2P, U1 MAX232_TID, U2 LM2937, U3 MAX874

Commit message: Commit Prueba Archivos Placa
Parts:
- removed C15: 0,1micF, SM1206
- removed C19: C, SM1206
- removed JP7, JP8: JUMPER, PIN_ARRAY_2X1
- removed U3: MAX874, maxim-8-SC70-5L
- added PIN_ARRAY_1: Val**, PIN_ARRAY_1, F.Cu at (106.9, 30.9)
- added PIN_ARRAY_1: Val**, PIN_ARRAY_1, F.Cu at (65.2, 75.5)
- added PIN_ARRAY_1: Val**, PIN_ARRAY_1, F.Cu at (68.0, 75.6)
- added PIN_ARRAY_1: Val**, PIN_ARRAY_1, F.Cu at (65.7, 39.5)
- added PIN_ARRAY_1: Val**, PIN_ARRAY_1, F.Cu at (69.2, 39.6)
- moved DB9FD 5.85 mm to (104.4, 62.9)
- moved 0,1micF1 4.19 mm to (75.0, 56.4), turned to 270 degrees
- moved 0,1micF5 3.51 mm to (89.8, 55.1), turned to 270 degrees
- moved JP1 3.50 mm to (90.9, 61.0), turned to 270 degrees
- moved J1 3.41 mm to (97.0, 24.2)
- moved C11 3.12 mm to (47.3, 25.3)
- moved 0,1micF2 3.02 mm to (73.8, 62.7), turned to 270 degrees
- moved C12 2.46 mm to (50.6, 25.5)
- moved JP2 2.39 mm to (95.1, 61.1), turned to 270 degrees
- moved C13 2.30 mm to (54.8, 25.1)
- moved C14 2.20 mm to (58.5, 25.0)
- moved JP3 1.86 mm to (91.4, 68.4)
- moved R10 1.28 mm to (63.2, 22.8)
Connections:
- +1 pad 11: (no net) -> N-000011
- +1 pad 12: (no net) -> N-000008
- +1 pad 3: N-000004 (its old number) -> N-000008
- +1 pad 6: N-000018 -> N-000055
- C1 pad 2: DGND -> GND
- C2 pad 2: DGND -> GND
- C3 pad 2: DGND -> GND
- C5 pad 2: DGND -> GND
- C6 pad 2: DGND -> GND
- C7 pad 1: N-000055 -> N-000054
- C7 pad 2: DGND -> GND
- C8 pad 1: N-000054 -> N-000053
- C8 pad 2: DGND -> GND
- DB9FD pad 2: (no net) -> N-000033
- DB9FD pad 3: (no net) -> N-000027
- DB9FD pad 7: (no net) -> N-000026
- DB9FD pad 8: (no net) -> N-000034
- JP9 pad 1: (no net) -> N-000032
- Prueba1 pad 2: (no net) -> GND
- R3 pad 2: N-000004 (its old number) -> N-000008
- R6 pad 2: N-000018 -> N-000055
- R7 pad 1: N-000055 -> N-000054
- R8 pad 1: N-000054 -> N-000053
- U1 pad 13: (no net) -> N-000026
- U1 pad 14: (no net) -> N-000034
- U1 pad 7: (no net) -> N-000033
- U1 pad 8: (no net) -> N-000027
- U2 pad GND@: (no net) -> GND
Routing:
- net DGND: track 84.9 -> 0.00 mm, vias 2 -> 0
- net +3.3V: track 18.2 -> 71.8 mm, vias 0 -> 2
- net N-000034: track 0.00 -> 47.9 mm
- net N-000027: track 0.00 -> 46.8 mm
- net N-000074: track 79.8 -> 123.3 mm, vias 2 -> 0
- net N-000033: track 0.00 -> 42.1 mm
- net N-000032: track 0.00 -> 39.6 mm
- net N-000026: track 0.00 -> 37.5 mm
- net N-000008: track 0.00 -> 37.2 mm
- net N-000013: track 45.6 -> 19.7 mm
- net N-000011: track 0.00 -> 23.0 mm
- net N-000018: track 15.6 -> 0.00 mm
- net N-000024: track 29.3 -> 44.6 mm, vias 2 -> 1
- net N-000004 (its old number): track 14.3 -> 0.00 mm
- net N-000060: track 12.4 -> 0.00 mm
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- added copper zone on B.Cu, net GND
- added copper zone on F.Cu, net GND
Other:
- net class +12v added: clearance 0.254, trace_width 0.54, via_dia 0.889, via_drill 0.635
- net class Default: trace_width 0.254 -> 0.54
- net class GND added: clearance 0.254, trace_width 0.54, via_dia 0.889, via_drill 0.635
- net class N-000009 added: clearance 0.254, trace_width 0.54, via_dia 0.889, via_drill 0.635

Commit message: Merge remote-tracking branch 'origin/master'
Conflicts:
	.gitignore
	Placa/prueba1.lst
	Source/fuentes/adc
	Source/fuentes/adc.#1
	Source/fuentes/adc.#2
	Source/fuentes/adc.#3
	Source/fuentes/adc.M51
	Source/fuentes/comunicacion.#1
	Source/fuentes/comunicacion.#3
	Source/fuentes/comunicacion.LST
	Source/fuentes/comunicacion.M51
	Source/fuentes/comunicacion.OBJ
	Source/fuentes/configurador.LST
	Source/fuentes/configurador.OBJ
	Source/fuentes/conversor.LST
	Source/fuentes/conversor.OBJ
	Source/fuentes/interfaz.LST
	Source/fuentes/interfaz.OBJ
	Source/fuentes/interrupciones.LST
	Source/fuentes/interrupciones.OBJ
	Source/fuentes/main.LST
	Source/fuentes/main.OBJ
	Source/fuentes/memoria.LST
	Source/fuentes/memoria.OBJ
	Source/test/test_comunicacion.LST
	Source/test/test_comunicacion.OBJ
	Source/test/test_global.LST
	Source/test/test_global.OBJ

commit onda
Parts:
- removed the PIN_ARRAY_1 at (65.2, 75.5)
- added PIN_ARRAY_1: Val**, PIN_ARRAY_1, F.Cu at (56.4, 75.3)
- added PIN_ARRAY_1: Val**, PIN_ARRAY_1, F.Cu at (63.0, 61.4)
- added PIN_ARRAY_1: Val**, PIN_ARRAY_1, F.Cu at (63.0, 64.2)
- added PIN_ARRAY_1: Val**, PIN_ARRAY_1, F.Cu at (62.9, 67.0)
- added PIN_ARRAY_1: Val**, PIN_ARRAY_1, F.Cu at (63.0, 69.8)
- moved PIN_ARRAY_1 8.84 mm to (59.2, 75.3)
Connections:
- +1 pad 11: N-000011 (its old number) -> N-000033
- +1 pad 12: N-000008 (its old number) -> N-000013
- +1 pad 13: (no net) -> N-000019
- +1 pad 14: (no net) -> N-000025
- +1 pad 15: (no net) -> N-000027
- +1 pad 16: (no net) -> N-000022
- +1 pad 18: N-000005 -> N-000020
- +1 pad 2: N-000047 -> N-000046
- +1 pad 24: N-000035 -> (no net)
- +1 pad 3: N-000008 (its old number) -> N-000048
- +1 pad 31: N-000016 -> N-000001
- +1 pad 32: N-000015 -> N-000002
- +1 pad 6: N-000055 -> N-000057
- +1 pad 7: N-000009 (its old number) -> N-000055
- C1 pad 2: GND -> DGND
- C16 pad 1: N-000038 -> N-000012
- C2 pad 1: N-000048 -> N-000047
- C2 pad 2: GND -> DGND
- C3 pad 1: N-000050 -> N-000049
- C3 pad 2: GND -> DGND
- C5 pad 1: N-000046 -> N-000041
- C5 pad 2: GND -> DGND
- C6 pad 1: N-000057 -> N-000058
- C6 pad 2: GND -> DGND
- C7 pad 1: N-000054 -> N-000056
- C7 pad 2: GND -> DGND
- C8 pad 1: N-000053 (its old number) -> N-000054
- C8 pad 2: GND -> DGND
- J1 pad 3: N-000014 (its old number) -> N-000015
- JP2 pad 1: N-000005 -> N-000020
- JP9 pad 1: N-000032 -> N-000003
- JP9 pad 3: N-000014 (its old number) -> N-000015
- PIN_ARRAY_1 pad 1: N-000008 (its old number) -> N-000013
- PWR1 pad 2: (no net) -> GND
- R10 pad 2: N-000038 -> N-000012
- R11 pad 2: N-000038 -> N-000012
- R12 pad 2: N-000038 -> N-000012
- R13 pad 1: N-000035 -> (no net)
- R2 pad 1: N-000048 -> N-000047
- R2 pad 2: N-000047 -> N-000046
- R3 pad 1: N-000050 -> N-000049
- R3 pad 2: N-000008 (its old number) -> N-000048
- R5 pad 1: N-000046 -> N-000041
- R6 pad 1: N-000057 -> N-000058
- R6 pad 2: N-000055 -> N-000057
- R7 pad 1: N-000054 -> N-000056
- R7 pad 2: N-000009 (its old number) -> N-000055
- R8 pad 1: N-000053 (its old number) -> N-000054
- U1 pad 1: N-000019 -> N-000052
- U1 pad 13: N-000026 -> N-000035
- U1 pad 14: N-000034 -> N-000032
- U1 pad 3: N-000020 -> N-000051
- U1 pad 4: N-000029 -> N-000050
- U1 pad 5: N-000028 -> N-000039
- U1 pad 6: N-000025 -> N-000038
- U1 pad 7: N-000033 -> N-000031
- U1 pad 8: N-000027 -> N-000037
- U2 pad GND@: GND -> (no net)
- U2 pad IN: N-000038 -> (no net)
Routing:
- net N-000034: track 47.9 -> 2.01 mm
- net N-000031: track 0.00 -> 40.4 mm
- net N-000008 (its old number): track 37.2 -> 0.00 mm
- net N-000003: track 0.00 -> 37.1 mm
- net N-000005: track 32.5 -> 0.00 mm
- net N-000020: track 4.73 -> 34.7 mm
- net N-000013: track 0.00 -> 27.5 mm
- net N-000014 (its old number): track 23.6 -> 0.00 mm
- net N-000011 (its old number): track 23.0 -> 0.00 mm
- net N-000022: track 0.00 -> 21.0 mm
- net N-000012: track 0.00 -> 20.6 mm
- net N-000009 (its old number): track 19.5 -> 0.00 mm
- net N-000015: track 5.80 -> 24.6 mm
- net N-000027: track 46.8 -> 63.0 mm
- net N-000046: track 6.95 -> 21.7 mm
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